File: base/base.kicad_pcb (KiCad board)
At the start: 2 copper layers, 0 parts

Commit message: Carrier: import nets, go 4-layer, fix netclass patterns
carrier.kicad_pcb (equivalent of Update PCB from Schematic):
- U1 fpid bga67-to-dip: -> carrier:
- 17 nets imported, all 101 pads assigned, matching the schematic
  netlist pad for pad
- 4 copper layers on a JLCPCB 1.6 mm 4-layer stackup
  (1 oz outer / 0.5 oz inner, 0.2104 prepreg / 1.065 core)
- GND pour moved off F.Cu to In1.Cu

U1 stays on B.Cu and J1 on F.Cu: F.Cu is the mating face.

Net class patterns: root-sheet local labels land on the board as
"/IO1", "/{slash}CE" and so on, so the documented "IO*" pattern matched
nothing and all 15 signal nets fell through to Default. Replaced with
"/*" -> Signal, which now resolves correctly. VCC and GND come from
power symbols, are global, and stay unprefixed.

base: 4 copper layers; net classes and patterns aligned with carrier,
which is what docs/HANDOFF.md already claimed was true.

DRC: 0 violations, 37 unconnected items (nothing routed yet).

Co-Authored-By: Claude Opus 5 <noreply@anthropic.com>
Other:
- copper layers 2 -> 4
Changed lines of the file:
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@@
 	(layers
 		(0 "F.Cu" signal)
+		(4 "In1.Cu" signal)
+		(6 "In2.Cu" signal)
 		(2 "B.Cu" signal)
 		(9 "F.Adhes" user "F.Adhesive")
