File: base/base.kicad_pcb (KiCad board)
At the start: 4 copper layers, 0 parts

Commit message: Finish base routing: 16 of 17 connections
tools/route_base.py is additive and re-runnable. It removes only its own
output -- vias and inner-layer tracks -- so Alex's F.Cu/B.Cu hand routing
survives a rerun, and it plans the whole board before committing anything so
a bad net ordering can be thrown away rather than hand-unpicked.

Routed: IO1-IO4, /RE, /ALE, /WP, /WE, /CE, VCC J1.10 and J2.12<->J2.37, and
R1's pull-up tail. Six of these sit on the wrong side of J1 -- IO1-IO4 are on
the odd row but land on the right-hand DIP column, /WE and /CE the reverse --
so they drop to In1/In2 and cross under the connector.

The zone was the reason every J1 GND pad read unconnected: it was on KiCad's
stock 0.5 mm clearance / 0.25 min width / 0.5 thermal gap, and a pour on those
settings cannot approach a 0.4 mm-pitch connector from any direction. Now on
the carrier's 0.2 / 0.15 / 0.3 with solid pad connection. 0.15 is load-bearing:
at 0.25 the pour needs 0.65 mm to reach a GND pad between two escape stubs and
has exactly 0.65, and all 13 go unconnected again.

Bugs found and fixed in my own checker along the way, each caught by DRC
rather than by reading the code:
  - pads were obstacles on every layer, so J1's B.Cu pads walled off both
    inner layers under the connector -- exactly the space the crossing nets
    need
  - track width was assumed 0.15, but Power-class runs are 0.4, under-
    reporting clearance to the VCC tracks by 0.125 mm
  - hole-to-hole was skipped for same-net pads and same-net vias, which
    stacked stitching vias on escape vias (18 holes_co_located)
  - the board edge was taken as a bounding box, but base's outline carries
    (radius 3), so stitching vias landed in corners that do not exist
  - strip() dropped its references to removed items, and pcbnew then freed
    them under the board; GetArea() started returning raw SwigPyObjects

DRC: no clearance, hole or edge violations, 0 unrouted signal nets.

Still open, both needing a decision rather than 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
Parts:
- added C1: 1uF, Capacitor_SMD:C_0603_1608Metric_Pad1.08x0.95mm_HandSolder, F.Cu at (112.0, 90.8)
- added C2: 100nF, Capacitor_SMD:C_0603_1608Metric_Pad1.08x0.95mm_HandSolder, F.Cu at (112.0, 89.0)
- added J1: DF40GB(1.5)-30DS-0.4V(51), Connector_Hirose_DF40:HIROSE_DF40GB-30DS-0.4V_51_, B.Cu at (124.1, 91.1)
- added J2: DIP-48_Socket, base:DIP-48_Socket_W15.24mm_P2.54mm, F.Cu at (116.5, 62.0)
- added R1: 10k, Resistor_SMD:R_0603_1608Metric_Pad0.98x0.95mm_HandSolder, F.Cu at (112.4, 77.3)
- added R2: 10k, Resistor_SMD:R_0603_1608Metric_Pad0.98x0.95mm_HandSolder, F.Cu at (111.6, 107.9)
Routing:
- net VCC: track 0.00 -> 154.7 mm, vias 0 -> 1
- net //WE: track 0.00 -> 129.8 mm
- net /RY//BY: track 0.00 -> 37.7 mm
- net //WP: track 0.00 -> 30.3 mm, vias 0 -> 1
- net /IO1: track 0.00 -> 30.2 mm, vias 0 -> 1
- net /IO2: track 0.00 -> 28.1 mm, vias 0 -> 1
- net /IO3: track 0.00 -> 22.7 mm, vias 0 -> 1
- net /IO8: track 0.00 -> 21.3 mm
- net /IO4: track 0.00 -> 21.3 mm, vias 0 -> 1
- net //RE: track 0.00 -> 20.7 mm, vias 0 -> 1
- net //CE: track 0.00 -> 20.6 mm, vias 0 -> 1
- net /ALE: track 0.00 -> 19.5 mm, vias 0 -> 1
- net /IO6: track 0.00 -> 17.9 mm
- net /IO7: track 0.00 -> 16.8 mm
- net /IO5: track 0.00 -> 12.6 mm
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- added copper zone on B.Cu, net GND
- added copper zone on F.Cu, net GND
- added copper zone on In1.Cu, net GND
- added copper zone on In2.Cu, net GND
Other:
- board outline added: 30 x 90 mm
